File: pcb/v1.0/mt-choc/mt-choc.kicad_sch (KiCad schematic)
At the start: 136 parts, among them SW1 SW_Push, SW10 SW_Push, SW11 SW_Push, SW12 SW_Push, SW13 SW_Push, SW14 SW_Push, SW15 SW_Push, SW16 SW_Push, SW17 SW_Push, SW18 SW_Push, SW19 SW_Push, SW2 SW_Push, SW20 SW_Push, SW21 SW_Push, SW22 SW_Push, SW23 SW_Push, SW24 SW_Push_Combo, SW25 SW_Push, SW26 SW_Push, SW27 SW_Push, SW28 SW_Push, SW29 SW_Push, SW3 SW_Push, SW30 SW_Push, SW31 SW_Push, SW32 SW_Push, SW33 SW_Push, SW34 SW_Push, SW35 SW_Push, SW36 SW_Push, SW37 SW_Push, SW38 SW_Push, SW39 SW_Push, SW4 SW_Push, SW40 SW_Push, SW41 SW_Push, SW42 SW_Push, SW43 SW_Push, SW44 SW_Push, SW45 SW_Push, SW46 SW_Push, SW47 SW_Push, SW48 SW_Push, SW49 SW_Push, SW5 SW_Push, SW50 SW_Push, SW51 SW_Push, SW52 SW_Push, SW53 SW_Push, SW54 SW_Push, SW55 SW_Push, SW56 SW_Push, SW57 SW_Push, SW58 SW_Push, SW59 SW_Push, SW6 SW_Push, SW60 SW_Push, SW61 SW_Push, SW62 SW_Push, SW63 SW_Push, SW64 SW_Push, SW7 SW_Push, SW8 SW_Push, SW9 SW_Push, U1 RP2040_LCD_1p28

Commit message: Update main PCB schematic and layout
- Rewire COL4 and COL12. Previously connected to GP23 and GP24 which are
  used for INT1 and INT2 of the IMU.
Connections:
- net COL10: now also U1.34 (GP22); no longer U1.32 (GP21)
- net COL11: now also U1.6 (GP2); no longer U1.34 (GP22)
- net COL12: now also U1.8 (GP3); no longer U1.36 (GP23)
- net COL4: now also U1.22 (GP16); no longer U1.21 (GP24)
- net COL5: now also U1.24 (GP17); no longer U1.22 (GP16)
- net COL6: now also U1.26 (GP18); no longer U1.24 (GP17)
- net COL7: now also U1.28 (GP19); no longer U1.26 (GP18)
- net COL8: now also U1.30 (GP20); no longer U1.28 (GP19)
- net COL9: now also U1.32 (GP21); no longer U1.30 (GP20)
- net ROW3: now also U1.15 (GP15); no longer U1.6 (GP2)
- net ROW4: now also U1.13 (GP14); no longer U1.8 (GP3)
- net ROW5: now also U1.11 (GP13); no longer U1.15 (GP15)
Other:
- note added: "Do Not Use IMU: GP6, GP7, GP23, GP24 LCD: GP8, GP9, GP10, GP11, GP12, GP25 BAT: GP29"
Changed lines of the file:
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@@
   (no_connect (at 119.38 168.275))
   (no_connect (at 76.2 158.115))
+  (no_connect (at 96.52 153.035))
   (no_connect (at 139.7 155.575))
   (no_connect (at 76.2 150.495))
@@
   (no_connect (at 119.38 163.195))
   (no_connect (at 119.38 165.735))
-  (no_connect (at 139.7 163.195))
   (no_connect (at 76.2 168.275))
   (no_connect (at 139.7 168.275))
@@
   (no_connect (at 139.7 150.495))
   (no_connect (at 76.2 147.955))
-  (no_connect (at 139.7 160.655))
   (no_connect (at 76.2 153.035))
   (no_connect (at 139.7 158.115))
   (no_connect (at 96.52 150.495))
+  (no_connect (at 76.2 170.815))
   (no_connect (at 139.7 153.035))
   (wire (pts (xy 27.305 46.99) (xy 42.545 46.99))
@@
     (effects (font (size 1.27 1.27) (thickness 0.254) bold) (justify right bottom))
   )
+  (text "Do Not Use\nIMU: GP6, GP7, GP23, GP24\nLCD: GP8, GP9, GP10, GP11, GP12, GP25\nBAT: GP29"
+    (at 50.165 193.04 0)
+    (effects (font (size 1.27 1.27)) (justify left bottom))
+  )
   (text "1.25u" (at 24.765 118.11 0)
     (effects (font (size 1.27 1.27) (thickness 0.254) bold) (justify right bottom))
@@
     )
   )
-  (global_label "COL10" (shape input) (at 96.52 158.115 0) (fields_autoplaced)
-    (effects (font (size 1.27 1.27)) (justify left))
-    (property "Intersheetrefs" "${INTERSHEET_REFS}" (at 104.9807 158.0356 0)
-      (effects (font (size 1.27 1.27)) (justify left) hide)
-    )
-  )
-  (global_label "COL9" (shape input) (at 96.52 160.655 0) (fields_autoplaced)
+  (global_label "COL10" (shape input) (at 96.52 155.575 0) (fields_autoplaced)
+    (effects (font (size 1.27 1.27)) (justify left))
+    (property "Intersheetrefs" "${INTERSHEET_REFS}" (at 104.9807 155.4956 0)
+      (effects (font (size 1.27 1.27)) (justify left) hide)
+    )
+  )
+  (global_label "COL9" (shape input) (at 96.52 158.115 0) (fields_autoplaced)
+    (effects (font (size 1.27 1.27)) (justify left))
+    (property "Intersheetrefs" "${INTERSHEET_REFS}" (at 103.7712 158.0356 0)
+      (effects (font (size 1.27 1.27)) (justify left) hide)
+    )
+  )
+  (global_label "ROW4" (shape input) (at 139.7 163.195 0) (fields_autoplaced)
+    (effects (font (size 1.27 1.27)) (justify left))
+    (property "Intersheetrefs" "${INTERSHEET_REFS}" (at 147.8672 163.195 0)
+      (effects (font (size 1.27 1.27)) (justify left) hide)
+    )
+  )
+  (global_label "ROW5" (shape input) (at 245.745 120.65 0) (fields_autoplaced)
+    (effects (font (size 1.27 1.27)) (justify left))
+    (property "Intersheetrefs" "${INTERSHEET_REFS}" (at 253.4195 120.5706 0)
+      (effects (font (size 1.27 1.27)) (justify left) hide)
+    )
+  )
+  (global_label "COL11" (shape input) (at 186.69 25.4 90) (fields_autoplaced)
+    (effects (font (size 1.27 1.27)) (justify left))
+    (property "Intersheetrefs" "${INTERSHEET_REFS}" (at 186.6106 16.9393 90)
+      (effects (font (size 1.27 1.27)) (justify left) hide)
+    )
+  )
+  (global_label "COL8" (shape input) (at 96.52 160.655 0) (fields_autoplaced)
     (effects (font (size 1.27 1.27)) (justify left))
     (property "Intersheetrefs" "${INTERSHEET_REFS}" (at 103.7712 160.5756 0)
@@
     )
   )
-  (global_label "ROW4" (shape input) (at 119.38 155.575 180) (fields_autoplaced)
+  (global_label "COL4" (shape input) (at 83.185 25.4 90) (fields_autoplaced)
+    (effects (font (size 1.27 1.27)) (justify left))
+    (property "Intersheetrefs" "${INTERSHEET_REFS}" (at 83.1056 18.1488 90)
+      (effects (font (size 1.27 1.27)) (justify left) hide)
+    )
+  )
+  (global_label "ROW3" (shape input) (at 245.745 83.82 0) (fields_autoplaced)
+    (effects (font (size 1.27 1.27)) (justify left))
+    (property "Intersheetrefs" "${INTERSHEET_REFS}" (at 253.4195 83.7406 0)
+      (effects (font (size 1.27 1.27)) (justify left) hide)
+    )
+  )
+  (global_label "COL11" (shape input) (at 119.38 153.035 180) (fields_autoplaced)
     (effects (font (size 1.27 1.27)) (justify right))
-    (property "Intersheetrefs" "${INTERSHEET_REFS}" (at 111.7055 155.4956 0)
+    (property "Intersheetrefs" "${INTERSHEET_REFS}" (at 110.4266 153.035 0)
       (effects (font (size 1.27 1.27)) (justify right) hide)
     )
   )
-  (global_label "ROW5" (shape input) (at 245.745 120.65 0) (fields_autoplaced)
-    (effects (font (size 1.27 1.27)) (justify left))
-    (property "Intersheetrefs" "${INTERSHEET_REFS}" (at 253.4195 120.5706 0)
-      (effects (font (size 1.27 1.27)) (justify left) hide)
-    )
-  )
-  (global_label "COL11" (shape input) (at 186.69 25.4 90) (fields_autoplaced)
-    (effects (font (size 1.27 1.27)) (justify left))
-    (property "Intersheetrefs" "${INTERSHEET_REFS}" (at 186.6106 16.9393 90)
-      (effects (font (size 1.27 1.27)) (justify left) hide)
-    )
-  )
-  (global_label "COL8" (shape input) (at 96.52 163.195 0) (fields_autoplaced)
-    (effects (font (size 1.27 1.27)) (justify left))
-    (property "Intersheetrefs" "${INTERSHEET_REFS}" (at 103.7712 163.1156 0)
-      (effects (font (size 1.27 1.27)) (justify left) hide)
-    )
-  )
-  (global_label "COL4" (shape input) (at 83.185 25.4 90) (fields_autoplaced)
-    (effects (font (size 1.27 1.27)) (justify left))
-    (property "Intersheetrefs" "${INTERSHEET_REFS}" (at 83.1056 18.1488 90)
-      (effects (font (size 1.27 1.27)) (justify left) hide)
-    )
-  )
-  (global_label "ROW3" (shape input) (at 245.745 83.82 0) (fields_autoplaced)
-    (effects (font (size 1.27 1.27)) (justify left))
-    (property "Intersheetrefs" "${INTERSHEET_REFS}" (at 253.4195 83.7406 0)
-      (effects (font (size 1.27 1.27)) (justify left) hide)
-    )
-  )
-  (global_label "COL11" (shape input) (at 96.52 155.575 0) (fields_autoplaced)
-    (effects (font (size 1.27 1.27)) (justify left))
-    (property "Intersheetrefs" "${INTERSHEET_REFS}" (at 104.9807 155.4956 0)
-      (effects (font (size 1.27 1.27)) (justify left) hide)
-    )
-  )
-  (global_label "COL12" (shape input) (at 96.52 153.035 0) (fields_autoplaced)
-    (effects (font (size 1.27 1.27)) (justify left))
-    (property "Intersheetrefs" "${INTERSHEET_REFS}" (at 104.9807 152.9556 0)
-      (effects (font (size 1.27 1.27)) (justify left) hide)
+  (global_label "COL12" (shape input) (at 119.38 155.575 180) (fields_autoplaced)
+    (effects (font (size 1.27 1.27)) (justify right))
+    (property "Intersheetrefs" "${INTERSHEET_REFS}" (at 110.4266 155.575 0)
+      (effects (font (size 1.27 1.27)) (justify right) hide)
     )
   )
@@
     )
   )
-  (global_label "COL5" (shape input) (at 96.52 170.815 0) (fields_autoplaced)
-    (effects (font (size 1.27 1.27)) (justify left))
-    (property "Intersheetrefs" "${INTERSHEET_REFS}" (at 103.7712 170.7356 0)
+  (global_label "COL5" (shape input) (at 96.52 168.275 0) (fields_autoplaced)
+    (effects (font (size 1.27 1.27)) (justify left))
+    (property "Intersheetrefs" "${INTERSHEET_REFS}" (at 103.7712 168.1956 0)
       (effects (font (size 1.27 1.27)) (justify left) hide)
     )
@@
     )
   )
-  (global_label "ROW3" (shape input) (at 119.38 153.035 180) (fields_autoplaced)
-    (effects (font (size 1.27 1.27)) (justify right))
-    (property "Intersheetrefs" "${INTERSHEET_REFS}" (at 111.7055 152.9556 0)
-      (effects (font (size 1.27 1.27)) (justify right) hide)
+  (global_label "ROW3" (shape input) (at 139.7 165.735 0) (fields_autoplaced)
+    (effects (font (size 1.27 1.27)) (justify left))
+    (property "Intersheetrefs" "${INTERSHEET_REFS}" (at 147.8672 165.735 0)
+      (effects (font (size 1.27 1.27)) (justify left) hide)
     )
   )
@@
     )
   )
-  (global_label "COL4" (shape input) (at 76.2 170.815 180) (fields_autoplaced)
-    (effects (font (size 1.27 1.27)) (justify right))
-    (property "Intersheetrefs" "${INTERSHEET_REFS}" (at 68.9488 170.7356 0)
-      (effects (font (size 1.27 1.27)) (justify right) hide)
+  (global_label "COL4" (shape input) (at 96.52 170.815 0) (fields_autoplaced)
+    (effects (font (size 1.27 1.27)) (justify left))
+    (property "Intersheetrefs" "${INTERSHEET_REFS}" (at 104.2639 170.815 0)
+      (effects (font (size 1.27 1.27)) (justify left) hide)
     )
   )
@@
     )
   )
-  (global_label "ROW5" (shape input) (at 139.7 165.735 0) (fields_autoplaced)
-    (effects (font (size 1.27 1.27)) (justify left))
-    (property "Intersheetrefs" "${INTERSHEET_REFS}" (at 147.3745 165.6556 0)
+  (global_label "ROW5" (shape input) (at 139.7 160.655 0) (fields_autoplaced)
+    (effects (font (size 1.27 1.27)) (justify left))
+    (property "Intersheetrefs" "${INTERSHEET_REFS}" (at 147.3745 160.5756 0)
       (effects (font (size 1.27 1.27)) (justify left) hide)
     )
@@
     )
   )
-  (global_label "COL7" (shape input) (at 96.52 165.735 0) (fields_autoplaced)
-    (effects (font (size 1.27 1.27)) (justify left))
-    (property "Intersheetrefs" "${INTERSHEET_REFS}" (at 103.7712 165.6556 0)
+  (global_label "COL7" (shape input) (at 96.52 163.195 0) (fields_autoplaced)
+    (effects (font (size 1.27 1.27)) (justify left))
+    (property "Intersheetrefs" "${INTERSHEET_REFS}" (at 103.7712 163.1156 0)
       (effects (font (size 1.27 1.27)) (justify left) hide)
     )
@@
     )
   )
-  (global_label "COL6" (shape input) (at 96.52 168.275 0) (fields_autoplaced)
-    (effects (font (size 1.27 1.27)) (justify left))
-    (property "Intersheetrefs" "${INTERSHEET_REFS}" (at 103.7712 168.1956 0)
-      (effects (font (size 1.27 1.27)) (justify left) hide)
-    )
+  (global_label "COL6" (shape input) (at 96.52 165.735 0) (fields_autoplaced)
+    (effects (font (size 1.27 1.27)) (justify left))
+    (property "Intersheetrefs" "${INTERSHEET_REFS}" (at 103.7712 165.6556 0)
+      (effects (font (size 1.27 1.27)) (justify left) hide)
+    )
